File: src/cmio.kicad_pcb (KiCad board)
At the start: 2 copper layers, 0 parts

Commit message: Some work on PCB
Signed-off-by: Mahyar Koshkouei <mahyar.koshkouei@gmail.com>
Parts:
- added C1: 4.7uF, Capacitors_SMD:C_0805_HandSoldering, F.Cu at (101.0, 99.4)
- added C10: 150uF, Capacitors_SMD:CP_Elec_6.3x7.7, F.Cu at (180.3, 52.1)
- added C11: 0.1uF, Capacitors_SMD:C_0805_HandSoldering, F.Cu at (89.4, 113.0)
- added C2: 4.7uF, Capacitors_SMD:C_0805_HandSoldering, F.Cu at (124.4, 109.0)
- added C3: 4.7uF, Capacitors_SMD:C_0805_HandSoldering, F.Cu at (109.2, 113.0)
- added C4: 4.7uF, Capacitors_SMD:C_0805_HandSoldering, F.Cu at (96.0, 99.4)
- added C5: 10nF, Capacitors_SMD:C_0805_HandSoldering, F.Cu at (104.2, 113.0)
- added C6: 4.7uF, Capacitors_SMD:C_0805_HandSoldering, F.Cu at (99.3, 113.0)
- added C7: 4.7uF, Capacitors_SMD:C_0805_HandSoldering, F.Cu at (94.3, 113.0)
- added C8: 0.1uF, Capacitors_SMD:C_0805_HandSoldering, F.Cu at (105.9, 99.4)
- added C9: 0.1uF, Capacitors_SMD:C_0805_HandSoldering, F.Cu at (119.5, 108.1)
- added J1: USB_POWER, foot:Micro_USB_B_10104110, F.Cu at (102.9, 91.4)
- added J2: BANK0, Pin_Headers:Pin_Header_Straight_2x20_Pitch2.54mm, F.Cu at (151.1, 91.4)
- added J3: USB_OTG, foot:Micro_USB_B_10104110, F.Cu at (90.2, 91.4)
- added J4: CM3Lite, foot:CM3_Socket_SODIMM_DDR1-2_TE_1612618_NoHole, B.Cu at (115.0, 82.5)
- added J5: TVOUT, foot:RCA_PHONO, F.Cu at (77.5, 91.4)
- added J6: BANK1, Pin_Headers:Pin_Header_Straight_2x10_Pitch2.54mm_SMD, F.Cu at (132.1, 77.5)
- added J7: Micro_SD_Card_TFP09_2_12B, foot:TFP09-2-12B, B.Cu at (135.9, 72.4)
- added L1: 2.2uH, Inductors_NEOSID:Neosid_Inductor_SM-NE29_SMD1008, F.Cu at (114.5, 109.6)
- added L2: 2.2uH, Inductors_NEOSID:Neosid_Inductor_SM-NE29_SMD1008, F.Cu at (187.5, 51.7)
- added R1: 100k, Resistors_SMD:R_0805_HandSoldering, F.Cu at (140.8, 99.4)
- added R2: 100k, Resistors_SMD:R_0805_HandSoldering, F.Cu at (182.9, 61.1)
- added R3: 200k, Resistors_SMD:R_0805_HandSoldering, F.Cu at (193.3, 50.2)
- added R4: 450k, Resistors_SMD:R_0805_HandSoldering, F.Cu at (145.9, 99.4)
- added R5: 10K, Resistors_SMD:R_0805_HandSoldering, F.Cu at (177.7, 61.1)
- added R6: 100K, Resistors_SMD:R_0805_HandSoldering, F.Cu at (140.8, 104.9)
- added R7: 100K, Resistors_SMD:R_0805_HandSoldering, F.Cu at (129.5, 108.9)
- added R8: 100K, Resistors_SMD:R_0805_HandSoldering, F.Cu at (177.7, 66.6)
- added R9: 100K, Resistors_SMD:R_0805_HandSoldering, F.Cu at (134.6, 106.6)
- added SW1: Reset, Buttons_Switches_SMD:SW_SPST_TL3342, F.Cu at (92.7, 82.5)
- added U1: AP3417B, TO_SOT_Packages_SMD:SOT-23-5_HandSoldering, F.Cu at (76.1, 112.9)
- added U2: AP3417B, TO_SOT_Packages_SMD:SOT-23-5_HandSoldering, F.Cu at (83.3, 112.9)
- added U3: SP6203EM5-L-2-8/TR, TO_SOT_Packages_SMD:SOT-23-5_HandSoldering, F.Cu at (102.8, 106.3)
- added U4: AP2401, Housings_SSOP:MSOP-8_3x3mm_Pitch0.65mm, F.Cu at (134.8, 100.3)

Commit message: Complete routing
Signed-off-by: Mahyar Koshkouei <mahyar.koshkouei@gmail.com>
Parts:
- removed J2: BANK0, Pin_Headers:Pin_Header_Straight_2x20_Pitch2.54mm
- added C12: 47uF, Capacitors_Tantalum_SMD:CP_Tantalum_Case-A_EIA-3216-18_Hand, F.Cu at (134.0, 101.0)
- added J8: Micro_SD_Card_TFP09_2_12B, foot:TFP09-2-12B, F.Cu at (169.8, 91.4)
- C10: value 150uF -> 47uF; footprint Capacitors_SMD:CP_Elec_6.3x7.7 -> Capacitors_Tantalum_SMD:CP_Tantalum_Case-A_EIA-3216-18_Hand
- J1: footprint foot:Micro_USB_B_10104110 -> foot:Molex_Right_Angle_SMT_TypeB_MicroUSB_105017
- J3: value USB_OTG -> BANK0; footprint foot:Micro_USB_B_10104110 -> Pin_Headers:Pin_Header_Straight_2x15_Pitch2.54mm
- J4: value CM3Lite -> USB_OTG; footprint foot:CM3_Socket_SODIMM_DDR1-2_TE_1612618_NoHole -> foot:Molex_Right_Angle_SMT_TypeB_MicroUSB_105017; moved to F.Cu
- J5: value TVOUT -> CM3Lite; footprint foot:RCA_PHONO -> foot:CM3_Socket_SODIMM_DDR1-2_TE_1612618_NoHole_NoEndSilkS; moved to B.Cu
- J6: value BANK1 -> TVOUT; footprint Pin_Headers:Pin_Header_Straight_2x10_Pitch2.54mm_SMD -> foot:RCA_PHONO
- J7: value Micro_SD_Card_TFP09_2_12B -> BANK1; footprint foot:TFP09-2-12B -> Pin_Headers:Pin_Header_Straight_2x10_Pitch2.54mm_SMD; moved to F.Cu
- R6, R7, R8, R9: moved to B.Cu
- moved J3 89.6 mm to (178.8, 104.6), turned to 270 degrees
- moved C11 85.1 mm to (172.7, 95.8)
- moved R3 83.0 mm to (118.4, 85.9)
- moved C10 78.0 mm to (117.3, 98.0), turned to 90 degrees
- moved L2 67.4 mm to (132.6, 90.8), turned to 90 degrees
- moved J5 66.2 mm to (143.5, 96.5), turned to 180 degrees
- moved R5 64.5 mm to (123.8, 96.5), turned to 180 degrees
- moved R2 56.7 mm to (138.7, 96.5)
- moved U2 53.7 mm to (134.0, 95.2), turned to 270 degrees
- moved U1 52.8 mm to (123.4, 89.4)
- moved C7 47.6 mm to (135.4, 88.9), turned to 90 degrees
- moved R7 44.9 mm to (168.3, 86.4)
- moved J6 36.8 mm to (106.7, 104.1), turned to 0 degrees
- moved J1 34.7 mm to (135.0, 104.4)
- moved J7 33.8 mm to (157.2, 98.6), turned to 270 degrees
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Connections:
- J3 pad 1: Net-(C10-Pad1) -> +3V3
- J3 pad 2: /D- -> GND
- J3 pad 3: /D+ -> /BCM_0
- J3 pad 4: OTGID -> /BCM_1
- J3 pad 5: GND -> /BCM_2
- J3 pad 6: GND -> /BCM_3
- J4 pad 1: GND -> Net-(C10-Pad1)
- J4 pad 2: (no net) -> /D-
- J4 pad 3: /BCM_0 -> /D+
- J4 pad 4: +3V3 -> OTGID
- J4 pad 5: /BCM_1 -> GND
- J5 pad 1: Net-(J4-Pad166) -> GND
- J5 pad 2: GND -> (no net)
- J6 pad 1: +3V3 -> Net-(J5-Pad166)
- J7 pad 1: DAT2 -> +3V3
- J7 pad 10: GND -> /BCM_35
- J7 pad 2: DAT3 -> GND
- J7 pad 3: CMD -> /BCM_28
- J7 pad 4: +3V3 -> /BCM_29
- J7 pad 5: CLK -> /BCM_30
- J7 pad 6: GND -> /BCM_31
- J7 pad 7: DAT0 -> /BCM_32
- J7 pad 8: DAT1 -> /BCM_33
- J7 pad 9: (no net) -> /BCM_34
- SW1 pad 2: Net-(J4-Pad177) -> Net-(J5-Pad177)
Routing:
- net GND: track 0.00 -> 127.4 mm, vias 0 -> 4
- net +3V3: track 0.00 -> 114.5 mm, vias 0 -> 3
- net +5V: track 0.00 -> 60.6 mm, vias 0 -> 2
- net Net-(J5-Pad177): track 0.00 -> 31.8 mm, vias 0 -> 3
- net /BCM_45: track 0.00 -> 19.2 mm, vias 0 -> 1
- net Net-(J5-Pad166): track 0.00 -> 18.5 mm, vias 0 -> 1
- net +2V8: track 0.00 -> 18.2 mm, vias 0 -> 1
- net OTGID: track 0.00 -> 17.5 mm, vias 0 -> 1
- net +1V8: track 0.00 -> 16.8 mm, vias 0 -> 1
- net /BCM_29: track 0.00 -> 15.9 mm, vias 0 -> 1
- net /BCM_44: track 0.00 -> 13.0 mm, vias 0 -> 1
- net /BCM_33: track 0.00 -> 10.7 mm, vias 0 -> 1
- net (no net): track 0.00 -> 10.5 mm
- net /BCM_35: track 0.00 -> 9.83 mm, vias 0 -> 1
- net /BCM_37: track 0.00 -> 9.53 mm, vias 0 -> 1
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- added copper zone on B.Cu, net +1V8
- added copper zone on F.Cu, net +1V8
- added copper zone on B.Cu, net +3V3
- added copper zone on B.Cu, net +5V
- added copper zone on F.Cu, net +5V
- added copper zone on B.Cu, net GND
- added copper zone on F.Cu, net GND
- added copper zone on F.Cu, net Net-(C10-Pad1)
- added copper zone on F.Cu, net Net-(L1-Pad1)
- added copper zone on F.Cu, net Net-(L2-Pad1)
Other:
- board outline added: 78.7 x 29.2 mm

Commit message: Add Board info to Silk Screen
Signed-off-by: Mahyar Koshkouei <mahyar.koshkouei@gmail.com>
Routing:
- net GND: track 127.4 -> 134.6 mm
Other:
- board text added: "Compute Module IO GNU GPL 3 Mahyar Koshkouei git.io/v5z7b"
- board text added: "Micro SD"
- board text added: "PWR"
- board text added: "RESET"
- board text added: "Raspberry Pi Compute Module (1/3/3L)"
- board text added: "USB"
Changed lines of the file:
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@@
     (area 104.089999 79.959999 182.930001 109.270001)
     (thickness 1.6)
-    (drawings 10)
-    (tracks 575)
+    (drawings 16)
+    (tracks 583)
     (zones 0)
     (modules 35)
@@
     (34 B.Paste user)
     (35 F.Paste user)
-    (36 B.SilkS user)
+    (36 B.SilkS user hide)
     (37 F.SilkS user)
     (38 B.Mask user)
@@
     (visible_elements FFFFFF7F)
     (pcbplotparams
-      (layerselection 0x00010_fffffffe)
+      (layerselection 0x01030_80000001)
       (usegerberextensions false)
-      (usegerberattributes true)
       (excludeedgelayer true)
       (linewidth 0.100000)
@@
       (padsonsilk false)
       (subtractmaskfromsilk false)
-      (outputformat 5)
+      (outputformat 1)
       (mirror false)
       (drillshape 0)
@@
     (tags "capacitor 0805")
     (attr smd)
-    (fp_text reference C7 (at 3.302 0 90) (layer F.SilkS)
+    (fp_text reference C7 (at 0 1.778 90) (layer F.SilkS)
       (effects (font (size 1 1) (thickness 0.15)))
     )
@@
     (pad 1 smd rect (at -1.14554 0 180) (size 1.02108 2.54) (layers F.Cu F.Paste F.Mask)
       (net 61 "Net-(L1-Pad1)"))
+    (model Inductors_SMD.3dshapes/L_0805.wrl
+      (at (xyz 0 0 0))
+      (scale (xyz 1 1 1))
+      (rotate (xyz 0 0 0))
+    )
   )
   (module Inductors_NEOSID:Neosid_Inductor_SM-NE29_SMD1008 (layer F.Cu)
@@
     (pad 2 smd rect (at 1.14554 0 90) (size 1.02108 2.54) (layers F.Cu F.Paste F.Mask)
       (net 3 +3V3))
+    (model Inductors_SMD.3dshapes/L_0805.wrl
+      (at (xyz 0 0 0))
+      (scale (xyz 1 1 1))
+      (rotate (xyz 0 0 0))
+    )
   )
   (module Resistors_SMD:R_0805_HandSoldering (layer F.Cu)
@@
       (net 2 GND))
     (model ${KISYS3DMOD}/Buttons_Switches_SMD.3dshapes/SW_SPST_TL3342.wrl
+      (at (xyz 0 0 0))
+      (scale (xyz 1 1 1))
+      (rotate (xyz 0 0 0))
+    )
+    (model Buttons_Switches_SMD.3dshapes/SW_SPST_EVQQ2_03W.wrl
       (at (xyz 0 0 0))
       (scale (xyz 1 1 1))
@@
     (pad "" np_thru_hole circle (at -33.4 0 180) (size 1.6 1.6) (drill 1.6) (layers *.Cu *.Mask))
   )
+  (gr_text "Compute Module IO\nGNU GPL 3\nMahyar Koshkouei\ngit.io/v5z7b" (at 159.512 85.344) (layer F.SilkS)
+    (effects (font (size 1.2 1.2) (thickness 0.25)) (justify right))
+  )
+  (gr_text "Raspberry Pi Compute Module (1/3/3L)" (at 143.51 82.55) (layer B.SilkS)
+    (effects (font (size 1.3 1.3) (thickness 0.25)) (justify mirror))
+  )
+  (gr_text RESET (at 111.76 82.804 90) (layer F.SilkS)
+    (effects (font (size 1 1) (thickness 0.15)))
+  )
+  (gr_text USB (at 114.554 107.188 90) (layer F.SilkS)
+    (effects (font (size 1 1) (thickness 0.15)))
+  )
+  (gr_text PWR (at 129.032 106.934 90) (layer F.SilkS)
+    (effects (font (size 1 1) (thickness 0.15)))
+  )
+  (gr_text "Micro SD" (at 180.34 84.074 90) (layer F.SilkS)
+    (effects (font (size 1 1) (thickness 0.15)))
+  )
   (gr_arc (start 104.648 108.712) (end 104.648 109.22) (angle 90) (layer Edge.Cuts) (width 0.1))
   (gr_arc (start 182.372 108.712) (end 182.88 108.712) (angle 90) (layer Edge.Cuts) (width 0.1))
@@
   (segment (start 125.175 96.52) (end 125.175 95.37) (width 0.5) (layer F.Cu) (net 1) (status 10))
   (segment (start 125.175 95.37) (end 123.531 93.726) (width 0.5) (layer F.Cu) (net 1))
+  (segment (start 150.2156 94.3864) (end 150.2156 95.6056) (width 0.25) (layer B.Cu) (net 2))
+  (segment (start 149.6568 93.8276) (end 150.2156 94.3864) (width 0.25) (layer B.Cu) (net 2))
+  (segment (start 149.6568 93.6732) (end 149.6568 93.8276) (width 0.25) (layer B.Cu) (net 2))
+  (segment (start 149.66 92.42) (end 149.66 93.67) (width 0.25) (layer B.Cu) (net 2))
+  (segment (start 149.66 93.67) (end 149.6568 93.6732) (width 0.25) (layer B.Cu) (net 2))
+  (segment (start 147.9804 93.7904) (end 147.9804 96.1136) (width 0.25) (layer B.Cu) (net 2))
+  (segment (start 147.86 92.42) (end 147.86 93.67) (width 0.25) (layer B.Cu) (net 2))
+  (segment (start 147.86 93.67) (end 147.9804 93.7904) (width 0.25) (layer B.Cu) (net 2))
   (segment (start 148.378498 90.7415) (end 149.2315 90.7415) (width 0.25) (layer B.Cu) (net 2))
   (segment (start 149.2315 90.7415) (end 149.66 91.17) (width 0.25) (layer B.Cu) (net 2))
